Commit message: robot last

File: models_env/plane.urdf (robot description, URDF)
Before this commit: robot plane, 1 links, 0 joints
Links:
- removed link planeLink
- added link floor, mass .0; collision box size=30 30 10; visual mesh filename=plane.obj scale=1 1 1

File: models_robot/cat.urdf (robot description, URDF)
Before this commit: robot Cat, 19 links, 18 joints
Links:
- link bl4_link: mass 0.01 -> 0.2; geometry collision sphere radius=0.01; visual sphere radius=0.01
- link br4_link: mass 0.01 -> 0.2; geometry collision sphere radius=0.01; visual sphere radius=0.01
- link fl4_link: mass 0.01 -> 0.2
- link fr4_link: mass 0.01 -> 0.2
Joints:
- joint bl1: origin xyz=-0.097 0.045 0 rpy=0 0 0 -> xyz=-0.118 0.045 0 rpy=0 0 0
- joint bl2: origin xyz=0 0.035 -0.025 rpy=0 0 0 -> xyz=0 0.045 -0.025 rpy=0 0 0
- joint br1: origin xyz=-0.097 -0.045 0 rpy=0 0 0 -> xyz=-0.118 -0.045 0 rpy=0 0 0
- joint br2: origin xyz=0 -0.035 -0.025 rpy=0 0 0 -> xyz=0 -0.045 -0.025 rpy=0 0 0
- joint fl1: origin xyz=0.097 0.045 0 rpy=0 0 0 -> xyz=0.118 0.045 0 rpy=0 0 0
- joint fl2: origin xyz=0 0.035 -0.025 rpy=0 0 0 -> xyz=0 0.045 -0.025 rpy=0 0 0
- joint fr1: origin xyz=0.097 -0.045 0 rpy=0 0 0 -> xyz=0.118 -0.045 0 rpy=0 0 0
- joint fr2: origin xyz=0 -0.035 -0.025 rpy=0 0 0 -> xyz=0 -0.045 -0.025 rpy=0 0 0
