Commit message: updated

File: models_robot/cat.urdf (robot description, URDF)
Before this commit: robot Cat, 19 links, 18 joints
Joints:
- joint bl3: limit lower=-3.14159265359 upper=0.174533 effort=100 velocity=100 -> lower=-3.14159265359 upper=0.0 effort=100 velocity=100
- joint br3: limit lower=-3.14159265359 upper=0.174533 effort=100 velocity=100 -> lower=-3.14159265359 upper=0.0 effort=100 velocity=100
- joint fl3: limit lower=-3.14159265359 upper=0.174533 effort=100 velocity=100 -> lower=-3.14159265359 upper=0.0 effort=100 velocity=100
- joint fr3: limit lower=-3.14159265359 upper=0.174533 effort=100 velocity=100 -> lower=-3.14159265359 upper=0.0 effort=100 velocity=100

Commit message: robot env update

File: models_robot/cat.urdf (robot description, URDF)
Before this commit: robot Cat, 19 links, 18 joints
Joints:
- joint bl1: limit lower=-0.698132 upper=0.698132 effort=100 velocity=100 -> lower=-0.398132 upper=0.698132 effort=100 velocity=100
- joint bl2: limit lower=-1.57079632679 upper=1.57079632679 effort=100 velocity=100 -> lower=-1.22173 upper=1.22173 effort=100 velocity=100
- joint br1: limit lower=-0.698132 upper=0.698132 effort=100 velocity=100 -> lower=-0.698132 upper=0.398132 effort=100 velocity=100
- joint br2: limit lower=-1.57079632679 upper=1.57079632679 effort=100 velocity=100 -> lower=-1.22173 upper=1.22173 effort=100 velocity=100
- joint fl1: limit lower=-0.698132 upper=0.698132 effort=100 velocity=100 -> lower=-0.398132 upper=0.698132 effort=100 velocity=100
- joint fl2: limit lower=-1.57079632679 upper=1.57079632679 effort=100 velocity=100 -> lower=-1.22173 upper=1.22173 effort=100 velocity=100
- joint fr1: limit lower=-0.698132 upper=0.698132 effort=100 velocity=100 -> lower=-0.698132 upper=0.398132 effort=100 velocity=100
- joint fr2: limit lower=-1.57079632679 upper=1.57079632679 effort=100 velocity=100 -> lower=-1.22173 upper=1.22173 effort=100 velocity=100

Commit message: models updated

File: models_robot/cat.urdf (robot description, URDF)
Before this commit: robot Cat, 19 links, 18 joints
Links:
- link bl1_link: geometry collision box size=0.02 0.041 0.041; visual box size=0.02 0.041 0.041
- link bl2_link: geometry collision box size=0.02 0.005 0.07; visual box size=0.02 0.005 0.07
- link bl3_link: geometry collision box size=0.01 0.005 0.07; visual box size=0.01 0.005 0.07
- link br1_link: geometry collision box size=0.02 0.041 0.041; visual box size=0.02 0.041 0.041
- link br2_link: geometry collision box size=0.02 0.005 0.07; visual box size=0.02 0.005 0.07
- link br3_link: geometry collision box size=0.01 0.005 0.07; visual box size=0.01 0.005 0.07
- link chassis: geometry collision box size=0.14 0.1 0.04; visual box size=0.14 0.1 0.04
- link fl1_link: geometry collision box size=0.02 0.041 0.041; visual box size=0.02 0.041 0.041
- link fl2_link: geometry collision box size=0.02 0.005 0.07; visual box size=0.02 0.005 0.07
- link fl3_link: geometry collision box size=0.01 0.005 0.07; visual box size=0.01 0.005 0.07
- link fr1_link: geometry collision box size=0.02 0.041 0.041; visual box size=0.02 0.041 0.041
- link fr2_link: geometry collision box size=0.02 0.005 0.07; visual box size=0.02 0.005 0.07
- link fr3_link: geometry collision box size=0.01 0.005 0.07; visual box size=0.01 0.005 0.07

Commit message: data updated

File: models_robot/cat.urdf (robot description, URDF)
Before this commit: robot Cat, 19 links, 18 joints
Links:
- link fl4_link: geometry collision sphere radius=0.01; visual sphere radius=0.01
- link fr4_link: geometry collision sphere radius=0.01; visual sphere radius=0.01

Commit message: env updated

File: models_robot/cat.urdf (robot description, URDF)
Before this commit: robot Cat, 19 links, 18 joints
Links:
- link bl2_link: geometry collision box size=0.02 0.005 0.1; visual box size=0.02 0.005 0.1
- link bl3_link: geometry collision box size=0.01 0.005 0.09; visual box size=0.01 0.005 0.09
- link bl4_link: mass 0.2 -> 0.01
- link br2_link: mass 0.07 -> 0.05; geometry collision box size=0.02 0.005 0.1; visual box size=0.02 0.005 0.1
- link br3_link: geometry collision box size=0.01 0.005 0.09; visual box size=0.01 0.005 0.09
- link br4_link: mass 0.2 -> 0.01
- link chassis: geometry collision box size=0.2 0.1 0.04; visual box size=0.2 0.1 0.04
- link fl2_link: geometry collision box size=0.02 0.005 0.1; visual box size=0.02 0.005 0.1
- link fl3_link: mass 0.05 -> 0.02; geometry collision box size=0.01 0.005 0.09; visual box size=0.01 0.005 0.09
- link fl4_link: mass 0.2 -> 0.01
- link fr2_link: geometry collision box size=0.02 0.005 0.1; visual box size=0.02 0.005 0.1
- link fr3_link: geometry collision box size=0.01 0.005 0.09; visual box size=0.01 0.005 0.09
- link fr4_link: mass 0.2 -> 0.01
Joints:
- joint bl1: origin xyz=-0.118 0.045 0 rpy=0 0 0 -> xyz=-0.115 0.052 0 rpy=0 0 0
- joint bl3: origin xyz=0 0.0 -0.07 rpy=0 0 0 -> xyz=0 0.0 -0.1 rpy=0 0 0
- joint bl4: origin xyz=0 0 -0.08 rpy=0 0 0 -> xyz=0 0 -0.1 rpy=0 0 0
- joint br1: origin xyz=-0.118 -0.045 0 rpy=0 0 0 -> xyz=-0.115 -0.052 0 rpy=0 0 0
- joint br3: origin xyz=0 0.0 -0.07 rpy=0 0 0 -> xyz=0 0.0 -0.1 rpy=0 0 0
- joint br4: origin xyz=0 0 -0.08 rpy=0 0 0 -> xyz=0 0 -0.1 rpy=0 0 0
- joint fl1: origin xyz=0.118 0.045 0 rpy=0 0 0 -> xyz=0.115 0.052 0 rpy=0 0 0
- joint fl3: origin xyz=0 0.0 -0.07 rpy=0 0 0 -> xyz=0 0.0 -0.1 rpy=0 0 0
- joint fl4: origin xyz=0 0 -0.08 rpy=0 0 0 -> xyz=0 0 -0.1 rpy=0 0 0
- joint fr1: origin xyz=0.118 -0.045 0 rpy=0 0 0 -> xyz=0.115 -0.052 0 rpy=0 0 0
- joint fr3: origin xyz=0 0.0 -0.07 rpy=0 0 0 -> xyz=0 0.0 -0.1 rpy=0 0 0
- joint fr4: origin xyz=0 0 -0.08 rpy=0 0 0 -> xyz=0 0 -0.1 rpy=0 0 0

Commit message: model updated

File: models_robot/cat.urdf (robot description, URDF)
Before this commit: robot Cat, 19 links, 18 joints
Links:
- link bl3_link: mass 0.05 -> 0.03
- link br2_link: mass 0.05 -> 0.07
- link br3_link: mass 0.05 -> 0.03
- link chassis: mass 0.4 -> 1.0
- link fl3_link: mass 0.02 -> 0.03
- link fr3_link: mass 0.05 -> 0.03

Commit message: robot model updated

File: models_robot/cat.urdf (robot description, URDF)
Before this commit: robot Cat, 19 links, 18 joints
Links:
- link bl1_link: mass 0.07 -> 0.14
- link bl2_link: mass 0.07 -> 0.02
- link br1_link: mass 0.07 -> 0.14
- link br2_link: mass 0.07 -> 0.02
- link fl1_link: mass 0.07 -> 0.14
- link fl2_link: mass 0.07 -> 0.02
- link fr1_link: mass 0.07 -> 0.14
- link fr2_link: mass 0.07 -> 0.02
Joints:
- joint bl1: origin xyz=-0.115 0.052 0 rpy=0 0 0 -> xyz=-0.1075 0.052 0 rpy=0 0 0
- joint bl2: origin xyz=0 0.045 -0.025 rpy=0 0 0 -> xyz=0 0.01 -0.02 rpy=0 0 0
- joint br1: origin xyz=-0.115 -0.052 0 rpy=0 0 0 -> xyz=-0.1075 -0.052 0 rpy=0 0 0
- joint br2: origin xyz=0 -0.045 -0.025 rpy=0 0 0 -> xyz=0 -0.01 -0.02 rpy=0 0 0
- joint fl1: origin xyz=0.115 0.052 0 rpy=0 0 0 -> xyz=0.1075 0.052 0 rpy=0 0 0
- joint fl2: origin xyz=0 0.045 -0.025 rpy=0 0 0 -> xyz=0 0.01 -0.02 rpy=0 0 0
- joint fr1: origin xyz=0.115 -0.052 0 rpy=0 0 0 -> xyz=0.1075 -0.052 0 rpy=0 0 0
- joint fr2: origin xyz=0 -0.045 -0.025 rpy=0 0 0 -> xyz=0 -0.01 -0.02 rpy=0 0 0

Commit message: balance evironment

File: models_robot/cat.urdf (robot description, URDF)
Before this commit: robot Cat, 19 links, 18 joints
Links:
- link bl1_link: geometry collision box size=0.05 0.041 0.04; visual box size=0.05 0.041 0.04
- link br1_link: geometry collision box size=0.05 0.041 0.04; visual box size=0.05 0.041 0.04
- link chassis: geometry collision box size=0.1 0.06 0.03; collision box size=0.16 0.1 0.04
- link fl1_link: geometry collision box size=0.05 0.041 0.04; visual box size=0.05 0.041 0.04
- link fr1_link: geometry collision box size=0.05 0.041 0.04; visual box size=0.05 0.041 0.04
Joints:
- joint bl2: origin xyz=0 0.01 -0.02 rpy=0 0 0 -> xyz=0 0.01 0.0 rpy=0 0 0
- joint br2: origin xyz=0 -0.01 -0.02 rpy=0 0 0 -> xyz=0 -0.01 0.0 rpy=0 0 0
- joint fl2: origin xyz=0 0.01 -0.02 rpy=0 0 0 -> xyz=0 0.01 0.0 rpy=0 0 0
- joint fr2: origin xyz=0 -0.01 -0.02 rpy=0 0 0 -> xyz=0 -0.01 0.0 rpy=0 0 0

Commit message: joints fix

File: models_robot/cat.urdf (robot description, URDF)
Before this commit: robot Cat, 19 links, 18 joints
Joints:
- joint bl2: origin xyz=0 0.01 0.0 rpy=0 0 0 -> xyz=0 0.02 0.0 rpy=0 0 0
- joint br2: origin xyz=0 -0.01 0.0 rpy=0 0 0 -> xyz=0 -0.02 0.0 rpy=0 0 0
- joint fl2: origin xyz=0 0.01 0.0 rpy=0 0 0 -> xyz=0 0.02 0.0 rpy=0 0 0
- joint fr2: origin xyz=0 -0.01 0.0 rpy=0 0 0 -> xyz=0 -0.02 0.0 rpy=0 0 0
